File: GurtMachine/GurtMachine.kicad_sch (KiCad schematic)
At the start: 55 parts, among them J1 USB_C_Receptacle_USB2.0_16P, J10 Conn_01x02, J11 Conn_01x04, J12 Conn_01x03, J13 Conn_01x03, J14 Conn_01x02, J15 Conn_01x02, J2 Conn_01x02, J3 Conn_01x02, J4 Conn_01x02, J5 Conn_01x02, J6 Conn_01x02, J7 Conn_01x02, J8 Conn_01x02, J9 Conn_01x02, U1 AP2114HA-3.3TRG1, U2 MCP73831-2-MC, X1 ESP32-S3-WROOM-1-N16R8

Commit message: gurt
Parts:
- removed J11: Conn_01x04, symbol Connector_Generic:Conn_01x04
- removed U1: AP2114HA-3.3TRG1, SOT-223_DIO, symbol 2026-10-07_23-46-19:AP2114HA-3.3TRG1
- added C7: 100n, symbol Device:C
- added J16: Conn_01x02, symbol Connector_Generic:Conn_01x02
- added J17: Conn_01x05, symbol Connector_Generic:Conn_01x05
- added L1: 0.47u, symbol Device:L
- added R22: 10k, symbol Device:R
- added R23: 91k, symbol Device:R
- added R24: 511k, symbol Device:R
- added U3: MAX17048G_T10, MAX17048G_T10:SON50P200X200X80-9N, symbol MAX17048G_T10:MAX17048G_T10
- added U4: TPS63802DLAR, TPS63802DLAR:VREG_TPS63802DLAR, symbol TPS63802DLAR:TPS63802DLAR
- C5: value 4.7u -> 10u
- C6: value 4.7u -> 22u
- R3: value 2k -> 5k
Connections:
- net +3.3V: now also J17.4 (Pin_4), R22.1, R24.2, U4.6 (VOUT)
- net GND: now also C7.2, J16.2 (Pin_2), J17.5 (Pin_5), R23.1, U3.1 (CTG), U3.4 (GND), U3.6 (QSTRT), U3.9 (EP), U4.2 (MODE), U4.3 (AGND), U4.8 (GND)
- net SDA: now reaches X1.19 (IO11)
- net SDA: now also J17.2 (Pin_2), U3.8 (SDA)
- net SCL: now reaches X1.20 (IO12)
- net SCL: now also J17.3 (Pin_3), U3.7 (SCL)
- net at X1.8 (IO15): now also J17.1 (Pin_1), R22.2
- net BAT+: now reaches BT1.1 (+), C5.1, U2.3 (V_{BAT}), U2.4 (V_{BAT})
- net BAT+: now also C7.1, J16.1 (Pin_1), U3.2 (CELL), U3.3 (VDD), U4.1 (EN), U4.10 (VIN)
- new net: R23.2, R24.1, U4.4 (FB)
- new net: L1.1, U4.7 (L2)
- new net: L1.2, U4.9 (L1)
- no-connect marks 21 -> 22
Other:
- moved on the sheet: BT1, C5, D10, D5, D9, J5, J6, J9, R12, R13, R14, R15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
